File: power_circuit.sch (KiCad schematic (older format))
At the start: 8 parts

Commit message: annotation number
Parts:
- gave numbers to parts that had none: 8
Changed lines of the file:
@@
 $EndDescr
 $Comp
-L Regulator_Linear:AMS1117-5.0 U?
+L Regulator_Linear:AMS1117-5.0 U1
 U 1 1 5FFC84D2
 P 2400 1300
-F 0 "U?" H 2400 1542 50  0000 C CNN
+F 0 "U1" H 2400 1542 50  0000 C CNN
 F 1 "AMS1117-5.0" H 2400 1451 50  0000 C CNN
 F 2 "Package_TO_SOT_SMD:SOT-223-3_TabPin2" H 2400 1500 50  0001 C CNN
@@
 $EndComp
 $Comp
-L power:+5V #PWR?
+L power:+5V #PWR0102
 U 1 1 5FFC84D8
 P 2800 1300
-F 0 "#PWR?" H 2800 1150 50  0001 C CNN
+F 0 "#PWR0102" H 2800 1150 50  0001 C CNN
 F 1 "+5V" H 2815 1473 50  0000 C CNN
 F 2 "" H 2800 1300 50  0001 C CNN
@@
 $EndComp
 $Comp
-L Device:Ferrite_Bead_Small FB?
+L Device:Ferrite_Bead_Small FB1
 U 1 1 5FFC84DE
 P 1400 1300
-F 0 "FB?" V 1550 1300 50  0000 C CNN
+F 0 "FB1" V 1550 1300 50  0000 C CNN
 F 1 "Ferrite_Bead_Small" V 1650 1300 50  0000 C CNN
 F 2 "Inductor_SMD:L_0603_1608Metric" V 1330 1300 50  0001 C CNN
@@
 $EndComp
 $Comp
-L Device:D_Small D?
+L Device:D_Small D1
 U 1 1 5FFC84E4
 P 1600 1300
-F 0 "D?" H 1600 1093 50  0000 C CNN
+F 0 "D1" H 1600 1093 50  0000 C CNN
 F 1 "D_Small" H 1600 1184 50  0000 C CNN
 F 2 "Diode_SMD:D_SOD-123" V 1600 1300 50  0001 C CNN
@@
 $EndComp
 $Comp
-L Device:C_Small C?
+L Device:C_Small C8
 U 1 1 5FFC84EA
 P 2800 1400
-F 0 "C?" H 2892 1446 50  0000 L CNN
+F 0 "C8" H 2892 1446 50  0000 L CNN
 F 1 "100n" H 2892 1355 50  0000 L CNN
 F 2 "Capacitor_SMD:C_0603_1608Metric" H 2800 1400 50  0001 C CNN
@@
 $EndComp
 $Comp
-L Device:C_Small C?
+L Device:C_Small C5
 U 1 1 5FFC84F0
 P 2000 1400
-F 0 "C?" H 1850 1450 50  0000 L CNN
+F 0 "C5" H 1850 1450 50  0000 L CNN
 F 1 "100n" H 1800 1350 50  0000 L CNN
 F 2 "Capacitor_SMD:C_0603_1608Metric" H 2000 1400 50  0001 C CNN
@@
 Connection ~ 2400 1600
 $Comp
-L power:GND #PWR?
+L power:GND #PWR0103
 U 1 1 5FFC84FF
 P 2400 1600
-F 0 "#PWR?" H 2400 1350 50  0001 C CNN
+F 0 "#PWR0103" H 2400 1350 50  0001 C CNN
 F 1 "GND" H 2405 1427 50  0000 C CNN
 F 2 "" H 2400 1600 50  0001 C CNN
@@
 $EndComp
 $Comp
-L Device:LED_Small D?
+L Device:LED_Small D2
 U 1 1 5FFC8505
 P 3100 1300
-F 0 "D?" H 3100 1093 50  0000 C CNN
+F 0 "D2" H 3100 1093 50  0000 C CNN
 F 1 "LED_PWR" H 3100 1184 50  0000 C CNN
 F 2 "LED_SMD:LED_0402_1005Metric" V 3100 1300 50  0001 C CNN
@@
 $EndComp
 $Comp
-L Device:R_Small R?
+L Device:R_Small R5
 U 1 1 5FFC850B
 P 3300 1400
-F 0 "R?" H 3359 1446 50  0000 L CNN
+F 0 "R5" H 3359 1446 50  0000 L CNN
 F 1 "2.2k" H 3359 1355 50  0000 L CNN
 F 2 "Resistor_SMD:R_0402_1005Metric" H 3300 1400 50  0001 C CNN
@@
 VBUS
 $Comp
-L Device:Fuse_Small F?
+L Device:Fuse_Small F1
 U 1 1 5FFC8518
 P 1800 1300
-F 0 "F?" H 1900 1500 50  0000 C CNN
+F 0 "F1" H 1900 1500 50  0000 C CNN
 F 1 "500mA" H 1900 1400 50  0000 C CNN
 F 2 "Fuse:Fuse_0603_1608Metric" H 1800 1300 50  0001 C CNN
@@
 5V Regulator
 $Comp
-L power:PWR_FLAG #FLG?
+L power:PWR_FLAG #FLG0101
 U 1 1 5FFC8523
 P 2000 1300
-F 0 "#FLG?" H 2000 1375 50  0001 C CNN
+F 0 "#FLG0101" H 2000 1375 50  0001 C CNN
 F 1 "PWR_FLAG" H 2000 1473 50  0000 C CNN
 F 2 "" H 2000 1300 50  0001 C CNN
