File: usb_ic.sch (KiCad schematic (older format))
At the start: 12 parts

Commit message: annotation number
Parts:
- gave numbers to parts that had none: 12
Changed lines of the file:
@@
 $EndDescr
 $Comp
-L Device:R_Small R?
+L Device:R_Small R3
 U 1 1 5FFE2B6B
 P 2350 2250
-F 0 "R?" V 2546 2250 50  0000 C CNN
+F 0 "R3" V 2546 2250 50  0000 C CNN
 F 1 "27" V 2455 2250 50  0000 C CNN
 F 2 "Resistor_SMD:R_0402_1005Metric" H 2350 2250 50  0001 C CNN
@@
 $EndComp
 $Comp
-L Device:R_Small R?
+L Device:R_Small R4
 U 1 1 5FFE2B71
 P 2350 2350
-F 0 "R?" V 2150 2350 50  0000 C CNN
+F 0 "R4" V 2150 2350 50  0000 C CNN
 F 1 "27" V 2250 2350 50  0000 C CNN
 F 2 "Resistor_SMD:R_0402_1005Metric" H 2350 2350 50  0001 C CNN
@@
 USB_DP
 $Comp
-L Device:C_Small C?
+L Device:C_Small C6
 U 1 1 5FFE2B7B
 P 2000 2350
-F 0 "C?" H 2092 2396 50  0000 L CNN
+F 0 "C6" H 2092 2396 50  0000 L CNN
 F 1 "47p" H 2092 2305 50  0000 L CNN
 F 2 "Capacitor_SMD:C_0402_1005Metric" H 2000 2350 50  0001 C CNN
@@
 $EndComp
 $Comp
-L Device:C_Small C?
+L Device:C_Small C4
 U 1 1 5FFE2B81
 P 1800 2450
-F 0 "C?" H 1892 2496 50  0000 L CNN
+F 0 "C4" H 1892 2496 50  0000 L CNN
 F 1 "47p" H 1892 2405 50  0000 L CNN
 F 2 "Capacitor_SMD:C_0402_1005Metric" H 1800 2450 50  0001 C CNN
@@
 $EndComp
 $Comp
-L power:GND #PWR?
+L power:GND #PWR0104
 U 1 1 5FFE2B87
 P 1800 2650
-F 0 "#PWR?" H 1800 2400 50  0001 C CNN
+F 0 "#PWR0104" H 1800 2400 50  0001 C CNN
 F 1 "GND" H 1805 2477 50  0000 C CNN
 F 2 "" H 1800 2650 50  0001 C CNN
@@
 USB IC
 $Comp
-L Device:LED_Small D?
+L Device:LED_Small D3
 U 1 1 5FFE2B9C
 P 2050 3000
-F 0 "D?" H 2050 2900 50  0000 C CNN
+F 0 "D3" H 2050 2900 50  0000 C CNN
 F 1 "LED_TX" H 2050 2950 50  0000 C CNN
 F 2 "LED_SMD:LED_0402_1005Metric" V 2050 3000 50  0001 C CNN
@@
 $EndComp
 $Comp
-L Device:LED_Small D?
+L Device:LED_Small D4
 U 1 1 5FFE2BA2
 P 2050 3100
-F 0 "D?" H 2050 3300 50  0000 C CNN
+F 0 "D4" H 2050 3300 50  0000 C CNN
 F 1 "LED_RX" H 2050 3200 50  0000 C CNN
 F 2 "LED_SMD:LED_0402_1005Metric" V 2050 3100 50  0001 C CNN
@@
 	2350 3100 2150 3100
 $Comp
-L Device:R_Small R?
+L Device:R_Small R1
 U 1 1 5FFE2BAE
 P 1850 3000
-F 0 "R?" H 1909 3046 50  0000 L CNN
+F 0 "R1" H 1909 3046 50  0000 L CNN
 F 1 "2.2k" H 1909 2955 50  0000 L CNN
 F 2 "Resistor_SMD:R_0402_1005Metric" H 1850 3000 50  0001 C CNN
@@
 $EndComp
 $Comp
-L Device:R_Small R?
+L Device:R_Small R2
 U 1 1 5FFE2BB4
 P 1850 3100
-F 0 "R?" H 1909 3146 50  0000 L CNN
+F 0 "R2" H 1909 3146 50  0000 L CNN
 F 1 "2.2k" H 1909 3055 50  0000 L CNN
 F 2 "Resistor_SMD:R_0402_1005Metric" H 1850 3100 50  0001 C CNN
@@
 Connection ~ 1450 3000
 $Comp
-L power:+5V #PWR?
+L power:+5V #PWR0105
 U 1 1 5FFE2BBF
 P 1450 2950
-F 0 "#PWR?" H 1450 2800 50  0001 C CNN
+F 0 "#PWR0105" H 1450 2800 50  0001 C CNN
 F 1 "+5V" H 1465 3123 50  0000 C CNN
 F 2 "" H 1450 2950 50  0001 C CNN
@@
 $EndComp
 $Comp
-L power:GND #PWR?
+L power:GND #PWR0106
 U 1 1 5FFE2BC5
 P 2600 3500
-F 0 "#PWR?" H 2600 3250 50  0001 C CNN
+F 0 "#PWR0106" H 2600 3250 50  0001 C CNN
 F 1 "GND" H 2605 3327 50  0000 C CNN
 F 2 "" H 2600 3500 50  0001 C CNN
@@
 $EndComp
 $Comp
-L Interface_USB:CP2104 U?
+L Interface_USB:CP2104 U3
 U 1 1 5FFE2BCB
 P 3300 2350
-F 0 "U?" H 3300 1261 50  0000 C CNN
+F 0 "U3" H 3300 1261 50  0000 C CNN
 F 1 "CP2104" H 3300 1170 50  0000 C CNN
 F 2 "Package_DFN_QFN:QFN-24-1EP_4x4mm_P0.5mm_EP2.6x2.6mm" H 3450 1400 50  0001 L CNN
@@
 $EndComp
 $Comp
-L Device:C_Small C?
+L Device:C_Small C10
 U 1 1 5FFE2BD1
 P 2600 3400
-F 0 "C?" H 2692 3446 50  0000 L CNN
+F 0 "C10" H 2692 3446 50  0000 L CNN
 F 1 "4.7u" H 2692 3355 50  0000 L CNN
 F 2 "Capacitor_SMD:C_0603_1608Metric" H 2600 3400 50  0001 C CNN
@@
 	2600 3300 2600 3050
 $Comp
-L power:+5V #PWR?
+L power:+5V #PWR0107
 U 1 1 5FFE2BD8
 P 2000 1450
-F 0 "#PWR?" H 2000 1300 50  0001 C CNN
+F 0 "#PWR0107" H 2000 1300 50  0001 C CNN
 F 1 "+5V" H 2015 1623 50  0000 C CNN
 F 2 "" H 2000 1450 50  0001 C CNN
@@
 $EndComp
 $Comp
-L Device:C_Small C?
+L Device:C_Small C9
 U 1 1 5FFE2BDE
 P 2000 1550
-F 0 "C?" H 2092 1596 50  0000 L CNN
+F 0 "C9" H 2092 1596 50  0000 L CNN
 F 1 "1u" H 2092 1505 50  0000 L CNN
 F 2 "Capacitor_SMD:C_0603_1608Metric" H 2000 1550 50  0001 C CNN
@@
 $EndComp
 $Comp
-L power:GND #PWR?
+L power:GND #PWR0108
 U 1 1 5FFE2BE4
 P 2000 1650
-F 0 "#PWR?" H 2000 1400 50  0001 C CNN
+F 0 "#PWR0108" H 2000 1400 50  0001 C CNN
 F 1 "GND" H 2005 1477 50  0000 C CNN
 F 2 "" H 2000 1650 50  0001 C CNN
@@
 Connection ~ 2600 3500
 $Comp
-L Device:R_Small R?
+L Device:R_Small R6
 U 1 1 5FFE2BF1
 P 4100 2850
-F 0 "R?" V 3904 2850 50  0000 C CNN
+F 0 "R6" V 3904 2850 50  0000 C CNN
 F 1 "4.7k" V 3995 2850 50  0000 C CNN
 F 2 "Resistor_SMD:R_0402_1005Metric" H 4100 2850 50  0001 C CNN
@@
 	0    1    1    0
 $EndComp
-Text GLabel 3100 1300 1    50   Input ~ 0
-VIO
-Text GLabel 4200 2850 2    50   Input ~ 0
-VIO
 Text GLabel 4000 2250 2    50   Input ~ 0
 UART_RXD
@@
 Wire Wire Line
 	3400 3350 3300 3350
-Wire Wire Line
-	3100 1300 3100 1450
 Connection ~ 3300 3350
 NoConn ~ 2600 2750
@@
 Wire Wire Line
 	2600 1450 2600 1750
+$Comp
+L power:+5V #PWR0109
+U 1 1 5FFB8D49
+P 4300 2850
+F 0 "#PWR0109" H 4300 2700 50  0001 C CNN
+F 1 "+5V" H 4315 3023 50  0000 C CNN
+F 2 "" H 4300 2850 50  0001 C CNN
+F 3 "" H 4300 2850 50  0001 C CNN
+	1    4300 2850
+	1    0    0    -1
+$EndComp
+Wire Wire Line
+	4300 2850 4200 2850
 $EndSCHEMATC

Commit message: Ready to order
Other:
- moved on the sheet: C10, C4, C6, C9, D3, D4, R1, R2, R3, R4, R6, U3
